Commit message: stl da mochila incluido no urdf

File: fsr_backpack_description/urdf/fsr_backpack.urdf.xacro (robot description, xacro)
@@ -41,6 +41,5 @@
 				<box size="0.0001 0.0001 0.0001" /> <!-- dimensoes apenas representativas -->
 			</geometry>
-			 <material
-				name="Gray">
+			 <material name="Gray">
 			<color
 			rgba="0.776470588235294 0.756862745098039 0.737254901960784 1" />
@@ -51,8 +50,11 @@
 	<link name="base_link">
 		<visual>
-			<origin xyz="0 0 0" rpy="0 0 0" />
-			<geometry>
-				<box size="0.1 0.1 0.1" />
-			</geometry>
+			<origin xyz="-0.20 0.18 -0.09" rpy="1.57 0 0" /> <!-- deslocamento entre desenho e TF (x = frente traz, y= lados, z=altura)-->
+			 <geometry>
+				<mesh filename="package://fsr_backpack_description/models/mochila.STL" scale=".0008 .0008 .0008"/>
+             </geometry>
+             <material name="mochila_material">
+				<color rgba="0.78 0.78 0.99 1" />
+			 </material>
 		</visual>
 	</link>
@@ -63,7 +65,7 @@
 	</joint>
 	<!-- IMU: MTi macro -->
-    <mti parent="base_link" x="0" y="0" z="0.25" rx="0" ry="0" rz="0" />
+    <mti parent="base_link" x="0.05" y="0" z="0.35" rx="3.14159" ry="0" rz="0" />
     <!-- GPS macro -->
-    <gps_antenna parent="base_link" x="0" y="-0.17" z="0.0" rx="0" ry="0" rz="0" />
+    <gps_antenna parent="base_link" x="0" y="0.0" z="0.40" rx="0" ry="0" rz="0" />
 	<!-- Camera
 	<link name="cam_pose">
