Commit message: updated version with data viewer

File: fsr_backpack_description/urdf/fsr_backpack_v0_5.urdf.xacro (robot description, xacro)
@@ -209,5 +209,5 @@
     <origin
       xyz="0 0 0"
-      rpy="0.21 2.7207E-18 0" />
+      rpy="0 2.7207E-18 0" />
     <parent
       link="arm_axel_link" />
@@ -262,6 +262,6 @@
 	k_velocity="0" />-->
   </joint>
-  <!-- Metal Detector Base    base_of_coil -->
-	<link name="metal_detector">
+  <!-- Metal Detector Base -->
+	<link name="base_of_coil">
 		<visual>
 			<origin xyz="0.13 -0.13 0" rpy="-0.37 3.1415 0" /> <!-- Deslocamento entre a TF e o desenho -->
@@ -277,9 +277,9 @@
 	<joint name="metal_detector_arm_joint" type="fixed">
 		<parent link="arm_elbow_up_down_link"/>
-		<child link="metal_detector" />
+		<child link="base_of_coil" />
 		<origin xyz="0 -1.30 -0.5" rpy="0 0 0" /> <!-- TF: distancia entre cotovelo e coil 1.3m abaixo e 0.5m pra frente -->
 	</joint>
 	<!-- Metal Detector Antena -->
-	<link name="metal_detector_middle_coil">
+	<link name="middle_coil">
 		<visual>
 			<origin xyz="0 0 0" rpy="0 0 0" /> <!-- Deslocamento entre a TF e o desenho -->
@@ -294,6 +294,6 @@
 	</link>
 	<joint name="metal_detector_coil_joint" type="fixed">
-		<parent link="metal_detector"/>
-		<child link="metal_detector_middle_coil" />
+		<parent link="base_of_coil"/>
+		<child link="middle_coil" />
 		<origin xyz="0 0 -0.08" rpy="0 0 0" /> <!-- TF: distancia entre base do detector e centro da coil -->
 	</joint>
