Commit message: urdf improved

File: fsr_backpack_description/urdf/fsr_backpack_parts/gps_antenna.urdf.xacro (robot description, xacro)
@@ -60,5 +60,5 @@
       				<origin xyz="-0.035 0 0" rpy="1.5708 0 0" />
       				<geometry>
-					<mesh filename="package://fsr_husky_description/models/fsr_husky_parts/gps_antenna.stl" />
+					<mesh filename="package://fsr_backpack_description/models/gps_antenna.stl" />
      			 	</geometry>
     			</collision>

File: fsr_backpack_description/urdf/fsr_backpack_v0_3.urdf.xacro (robot description, xacro)
@@ -50,10 +50,10 @@
 	<link name="base_link">
 		<visual>
-			<origin xyz="-0.22 0.22 -0.18" rpy="1.57 0 0" /> <!-- deslocamento entre desenho e TF (x = frente traz, y= lados, z=altura)-->
+			<origin xyz="-0.20 0.18 -0.09" rpy="1.57 0 0" /> <!-- deslocamento entre desenho e TF (x = frente traz, y= lados, z=altura)-->
 			 <geometry>
-				<mesh filename="package://fsr_backpack_description/models/mochila.STL" scale=".001 .001 .001"/>
+				<mesh filename="package://fsr_backpack_description/models/mochila.STL" scale=".0008 .0008 .0008"/>
              </geometry>
              <material name="mochila_material">
-				<color rgba="0.4 0.4 0.4 1" />
+				<color rgba="0.78 0.78 0.99 1" />
 			 </material>
 		</visual>
@@ -65,7 +65,7 @@
 	</joint>
 	<!-- IMU: MTi macro -->
-    <mti parent="base_link" x="0.10" y="0" z="0.39" rx="3.14159" ry="0" rz="0" />
+    <mti parent="base_link" x="0.05" y="0" z="0.35" rx="3.14159" ry="0" rz="0" />
     <!-- GPS macro -->
-    <gps_antenna parent="base_link" x="0.10" y="0.0" z="0.42" rx="0" ry="0" rz="0" />
+    <gps_antenna parent="base_link" x="0" y="0.0" z="0.40" rx="0" ry="0" rz="0" />
 	<!-- Camera
 	<link name="cam_pose">
@@ -82,8 +82,21 @@
 		<origin xyz="0 0 -0.25" rpy="0 1.57 0" />
 	</joint> -->
+	 <!-- <link name="gps_antenna">
+		<visual>
+			<origin xyz="0 0 0" rpy="0 0 0" />
+			<geometry>
+				<box size="0.001 0.001 0.001" />
+			</geometry>
+		</visual>
+	</link>
+	<joint name="gps_joint" type="fixed">
+		<parent link="base_link"/>
+		<child link="gps_antenna"/>
+		<origin xyz="0 -0.45 0.25" rpy="0 0 0" />
+	</joint> -->
 	<joint name="arm_base_link_joint" type="fixed">
 		<parent link="base_link"/>
 		<child link="arm_base_link"/>
-		<origin xyz="-0.1 0.25 0.25" rpy="0 0 0" /> <!-- ombro fica a 10cm para frente, 20cm ao lado e 25cm a cima do centro -->
+		<origin xyz="-0.1 0.20 0.25" rpy="0 0 0" /> <!-- ombro fica a 10cm para frente, 20cm ao lado e 25cm a cima do centro -->
 	</joint>
 	<!-- arm  -->
@@ -262,39 +275,27 @@
 	k_velocity="0" />-->
   </joint>
-  <!-- Metal Detector Base -->
-	<link name="base_of_coil">
-		<visual>
-			<origin xyz="0.13 -0.13 0" rpy="-0.37 3.1415 0" /> <!-- Deslocamento entre a TF e o desenho -->
+	<!-- Metal Detector Antena -->
+	<link name="middle_coil">
+		<visual>
+			<origin xyz="0.1 -0.1 0" rpy="-0.37 3.1415 0" /> <!-- Deslocamento entre a TF e o desenho -->
+			<!--
+			<geometry>
+				<box size="0.1 0.01 0.1" />
+			</geometry>
+			<material
+				name="DarkGray">
+			<color
+				rgba="0.776470588235294 0.756862745098039 0.737254901960784 1" />
+			</material> -->
 			 <geometry>
-				<mesh filename="package://fsr_backpack_description/models/Schiebel.STL" scale=".001 .001 .001"/>
+				<mesh filename="package://fsr_backpack_description/models/Schiebel.STL" scale=".0008 .0008 .0008"/>
             </geometry>
-            <material name="DarkGreen1">
-            <color
-				rgba="0 0.4 0 1" />
-			</material>
+            <material name="DarkGray" />
 		</visual>
 	</link>
 	<joint name="metal_detector_arm_joint" type="fixed">
 		<parent link="arm_elbow_up_down_link"/>
-		<child link="base_of_coil" />
-		<origin xyz="0 -1.30 -0.5" rpy="0 0 0" /> <!-- TF: distancia entre cotovelo e coil 1.3m abaixo e 0.5m pra frente -->
-	</joint>
-	<!-- Metal Detector Antena -->
-	<link name="middle_coil">
-		<visual>
-			<origin xyz="0 0 0" rpy="0 0 0" /> <!-- Deslocamento entre a TF e o desenho -->
-			<geometry>
-				<box size="0.01 0.01 0.01" />
-			</geometry>
-            <material name="Red">
-            <color
-				rgba="1 0 0 1" />
-			</material>
-		</visual>
-	</link>
-	<joint name="metal_detector_coil_joint" type="fixed">
-		<parent link="base_of_coil"/>
 		<child link="middle_coil" />
-		<origin xyz="0 0 -0.08" rpy="0 0 0" /> <!-- TF: distancia entre base do detector e centro da coil -->
+		<origin xyz="0 -1.3 -0.5" rpy="0 0 0" /> <!-- TF: distancia entre ombro e coil 1.3m abaixo e 0.5m pra frente -->
 	</joint>
 	<!-- Liga a joint a um "actuator name" -->

File: fsr_backpack_description/urdf/fsr_backpack_v0_4.urdf.xacro (robot description, xacro)
@@ -67,5 +67,5 @@
     <mti parent="base_link" x="0.10" y="0" z="0.39" rx="3.14159" ry="0" rz="0" />
     <!-- GPS macro -->
-    <gps_antenna parent="base_link" x="0.10" y="0.0" z="0.42" rx="0" ry="0" rz="0" />
+    <gps_antenna parent="base_link" x="0.10" y="0.0" z="0.43" rx="0" ry="0" rz="0" />
 	<!-- Camera
 	<link name="cam_pose">
@@ -81,4 +81,17 @@
 		<child link="cam_pose"/>
 		<origin xyz="0 0 -0.25" rpy="0 1.57 0" />
+	</joint> -->
+	 <!-- <link name="gps_antenna">
+		<visual>
+			<origin xyz="0 0 0" rpy="0 0 0" />
+			<geometry>
+				<box size="0.001 0.001 0.001" />
+			</geometry>
+		</visual>
+	</link>
+	<joint name="gps_joint" type="fixed">
+		<parent link="base_link"/>
+		<child link="gps_antenna"/>
+		<origin xyz="0 -0.45 0.25" rpy="0 0 0" />
 	</joint> -->
 	<joint name="arm_base_link_joint" type="fixed">
@@ -262,8 +275,8 @@
 	k_velocity="0" />-->
   </joint>
-  <!-- Metal Detector Base -->
-	<link name="base_of_coil">
-		<visual>
-			<origin xyz="0.13 -0.13 0" rpy="-0.37 3.1415 0" /> <!-- Deslocamento entre a TF e o desenho -->
+	<!-- Metal Detector Antena -->
+	<link name="middle_coil">
+		<visual>
+			<origin xyz="0.13 -0.1 0" rpy="-0.37 3.1415 0" /> <!-- Deslocamento entre a TF e o desenho -->
 			 <geometry>
 				<mesh filename="package://fsr_backpack_description/models/Schiebel.STL" scale=".001 .001 .001"/>
@@ -277,24 +290,6 @@
 	<joint name="metal_detector_arm_joint" type="fixed">
 		<parent link="arm_elbow_up_down_link"/>
-		<child link="base_of_coil" />
-		<origin xyz="0 -1.30 -0.5" rpy="0 0 0" /> <!-- TF: distancia entre cotovelo e coil 1.3m abaixo e 0.5m pra frente -->
-	</joint>
-	<!-- Metal Detector Antena -->
-	<link name="middle_coil">
-		<visual>
-			<origin xyz="0 0 0" rpy="0 0 0" /> <!-- Deslocamento entre a TF e o desenho -->
-			<geometry>
-				<box size="0.01 0.01 0.01" />
-			</geometry>
-            <material name="Red">
-            <color
-				rgba="1 0 0 1" />
-			</material>
-		</visual>
-	</link>
-	<joint name="metal_detector_coil_joint" type="fixed">
-		<parent link="base_of_coil"/>
 		<child link="middle_coil" />
-		<origin xyz="0 0 -0.08" rpy="0 0 0" /> <!-- TF: distancia entre base do detector e centro da coil -->
+		<origin xyz="0 -1.3 -0.5" rpy="0 0 0" /> <!-- TF: distancia entre cotovelo e coil 1.3m abaixo e 0.5m pra frente -->
 	</joint>
 	<!-- Liga a joint a um "actuator name" -->
